Commit message: Global scripts update and cosmetic changes (add floor)

File: urdf/object_point.urdf (robot description, URDF)
Before this commit: robot object, 1 links, 0 joints
Links:
- added link l_square; visual box size=0.03 0.03 0.02
- link base_link: geometry collision cylinder length=0.4 radius=0.01; visual cylinder length=0.4 radius=0.01
Joints:
- added joint j_object_one: type fixed, parent base_link, child l_square, origin xyz=0 0 0 rpy=0 0 0

File: urdf/obstacles_concaves.urdf (robot description, URDF)
Before this commit: robot obstacles, 14 links, 13 joints
Links:
- added link l_object_floor; visual box size=10 10 0.01
Joints:
- added joint j_object_floor: type fixed, parent obstacle_base, child l_object_floor, origin xyz=0 0 0 rpy=0 0 0

Commit message: Update of files from last paper submissions:
* remove obstacle colors
* add convenient functions in matplotlib library (as plotObstacles)
* update script to TADR2, add convergence graphs

File: urdf/object_point.urdf (robot description, URDF)
Before this commit: robot object, 2 links, 1 joints
Links:
- removed link l_square
- link base_link: geometry collision cylinder length=0.4 radius=0.02; visual cylinder length=0.4 radius=0.02
Joints:
- removed joint j_object_one

File: urdf/obstacles_concaves.urdf (robot description, URDF)
Before this commit: robot obstacles, 15 links, 14 joints
Links:
- removed link l_object_floor
Joints:
- removed joint j_object_floor
